File: 3 Wire EEG-test/3 Wire EEG/3 Wire EEG.kicad_sch (KiCad schematic)
At the start: 10 parts, among them J2 Electrode, J3 Conn_01x03_Pin

Commit message: Added from Pippa
Parts:
- removed J2: Electrode, symbol Connector:Conn_01x01_Pin
- removed J3: Conn_01x03_Pin, symbol Connector:Conn_01x03_Pin
- added J1: Signal, symbol Connector:Conn_01x01_Pin
- C1: renamed from CPow1; value 10nF -> C
- C2: renamed from C_HF_LP1; value 100pF -> C
- C3: renamed from C_HF_LP2; value 100pF -> C
- R1: renamed from R_pow_prot1; value 100 -> R
- R2: renamed from R-Decoupling1; value 100 -> R
- R3: renamed from R_User_Prot1; value 200K -> R
- R4: renamed from R2; value 10K -> R
- renumbered TLC272 to U2
Connections:
- net AVSS renamed GNDA
- net Signal: no longer names the net of R2.2
- net Signal: now also J1.1 (Pin_1)
Other:
- moved on the sheet: C1, C2, R4
